File: mariposa.kicad_pcb (KiCad board)
At the start: 2 copper layers, 52.1 x 109 mm, 53 parts, among them J1 Conn_01x22_Shielded, J2 Conn_01x03_MountingPin, J3 Conn_ARM_SWD_TagConnect_TC203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, J4 USB_C_Receptacle_USB2.0_16P, J5 Conn_02x03_Counter_Clockwise, J6 Conn_01x05_Socket, SW1 SW_Push, SW2 Slide_DPDT_SS22D06, SW3 SW_Push, U2 TPS7A0333PDBVR, U3 MCP73831T-2ACI/OT

Commit message: mariposa v2 RC2
Parts:
- removed D7, D8: LED, LED_SMD:LED_0805_2012Metric
- removed JP2, JP3, JP4: SolderJumper_2_Open, Jumper:SolderJumper-2_P1.3mm_Open_TrianglePad1.0x1.5mm
- removed R11: 20k, Resistor_SMD:R_0603_1608Metric
- removed R12: 12k, Resistor_SMD:R_0603_1608Metric
- removed RN1: 2x R22, PCM_Resistor_SMD_AKL:R_Array_Convex_2x0402
- added C1: 560pF, Capacitor_SMD:C_0603_1608Metric, B.Cu at (143.7, 88.0)
- added C2: 1uF, Capacitor_SMD:C_0603_1608Metric, B.Cu at (154.3, 91.2)
- added C3: 1uF, Capacitor_SMD:C_0603_1608Metric, B.Cu at (153.4, 93.6)
- added C4: 10nF, Capacitor_SMD:C_0402_1005Metric, B.Cu at (154.8, 51.0)
- added C5: 10nF, Capacitor_SMD:C_0402_1005Metric, B.Cu at (154.8, 56.0)
- added FB3: 240 Ohm, PCM_Ferrite_SMD_AKL:Ferrite_0603_1608Metric, B.Cu at (152.7, 91.2)
- added FB4: 240 Ohm, PCM_Ferrite_SMD_AKL:Ferrite_0603_1608Metric, B.Cu at (157.3, 88.3)
- added FB5: 120 Ohm, PCM_Ferrite_SMD_AKL:Ferrite_0805_2012Metric, B.Cu at (146.8, 53.5)
- added FB6: 240 Ohm, PCM_Ferrite_SMD_AKL:Ferrite_0603_1608Metric, B.Cu at (131.1, 68.4)
- added FB7: 240 Ohm, PCM_Ferrite_SMD_AKL:Ferrite_0603_1608Metric, B.Cu at (129.1, 65.8)
- added J7: Ext VCC Out, Connector_JST:JST_SUR_SM02B-SURS-TF_1x02-1MP_P0.80mm_Horizontal, B.Cu at (134.6, 72.3)
- added R13: 10k, Resistor_SMD:R_0603_1608Metric, B.Cu at (157.1, 86.7)
- added R5: 10k, Resistor_SMD:R_0603_1608Metric, B.Cu at (143.7, 91.1)
- added R6: 10k, Resistor_SMD:R_0603_1608Metric, B.Cu at (143.7, 85.0)
- added TP1: TestPoint, TestPoint:TestPoint_Pad_D1.0mm, B.Cu at (162.5, 135.9)
- added TP2: TestPoint, TestPoint:TestPoint_Pad_D1.0mm, B.Cu at (162.5, 133.9)
- added TP3: TestPoint, TestPoint:TestPoint_Pad_D1.0mm, B.Cu at (168.8, 103.5)
- added TP4: TestPoint, TestPoint:TestPoint_Pad_D1.0mm, B.Cu at (156.2, 80.8)
- added TP5: TestPoint, TestPoint:TestPoint_Pad_D1.0mm, B.Cu at (161.1, 119.2)
- added TP6: TestPoint, TestPoint:TestPoint_Pad_D1.0mm, B.Cu at (146.4, 92.8)
- added TP7: TestPoint, TestPoint:TestPoint_Pad_D1.0mm, B.Cu at (146.4, 90.7)
- added TP8: TestPoint, TestPoint:TestPoint_Pad_D1.0mm, B.Cu at (146.4, 94.9)
- BT1: footprint Connector_JST:JST_PH_S2B-PH-SM4-TB_1x02-1MP_P2.00mm_Horizontal -> Connector_JST:JST_GH_SM02B-GHS-TB_1x02-1MP_P1.25mm_Horizontal
- C46, C47: footprint Capacitor_SMD:C_0805_2012Metric -> Capacitor_SMD:C_0603_1608Metric
- D5, D6: footprint LED_SMD:LED_0805_2012Metric -> LED_SMD:LED_1206_3216Metric_ReverseMount_Hole1.8x2.4mm
- FB1, FB2: value 60ohm -> 120 Ohm
- J2: footprint Connector_JST:JST_PH_S3B-PH-SM4-TB_1x03-1MP_P2.00mm_Horizontal -> Connector_JST:JST_SH_SM03B-SRSS-TB_1x03-1MP_P1.00mm_Horizontal
- J6: value Conn_01x05_Socket -> Conn_01x10_MountingPin; footprint coquette_footprints:5-pin horizontal display -> Connector_FFC-FPC:Hirose_FH12-10S-0.5SH_1x10-1MP_P0.50mm_Horizontal; moved to B.Cu
- R1, R8: footprint Resistor_SMD:R_0805_2012Metric -> Resistor_SMD:R_0603_1608Metric
- R2, R7: value 3k -> 2k
- moved D6 74.4 mm to (170.9, 39.6), turned to 180 degrees
- moved D5 74.4 mm to (129.1, 39.6), turned to 0 degrees
- moved R7 71.1 mm to (167.2, 40.3), turned to 180 degrees
- moved R2 71.1 mm to (132.9, 40.3), turned to 0 degrees
- moved D12 55.8 mm to (141.0, 50.7), turned to 180 degrees
- moved D11 46.3 mm to (150.0, 91.5)
- moved J6 45.0 mm to (150.0, 86.5)
- moved U2 38.5 mm to (157.6, 63.6)
- moved C44 38.1 mm to (157.4, 60.9)
- moved C45 37.5 mm to (156.6, 67.2), turned to -90 degrees
- moved SW2 34.0 mm to (165.4, 51.3), turned to -49 degrees
- moved D4 25.9 mm to (152.9, 66.1), turned to 0 degrees
- moved D45 17.2 mm to (152.9, 63.2), turned to 180 degrees
- moved D88 17.0 mm to (154.3, 59.0), turned to 90 degrees
- moved J3 12.5 mm to (162.0, 123.1), turned to -90 degrees
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Connections:
- net row_e renamed ch5
- C44 pad 1: Net-(D45-K) -> VDC
- D10 pad 1: /power/IN_D- -> gpio1
- D10 pad 3: /power/IN_D+ -> D-
- D10 pad 4: gpio2 -> D+
- D10 pad 6: gpio1 -> gpio2
- D11 pad 3: mosi -> cs
- D11 pad 6: cs -> mosi
- D12 pad 1: gpio4 -> status_led_2
- D12 pad 3: gpio3 -> sda
- D12 pad 6: sda -> status_led_1
- D13 pad 1: swdclk -> VDD
- D13 pad 4: reset -> swdclk
- D13 pad 6: led_data -> reset
- D45 pad 1: Net-(D45-K) -> VDC
- D88 pad 1: Net-(D45-K) -> VDC
- D9 pad 2: VBUS -> Net-(C4--)
- FB1 pad 1: Net-(FB1-Pad1) -> Net-(C4--)
- J1 pad 10: c4 -> ch10
- J1 pad 11: c3 -> ch11
- J1 pad 12: c2 -> ch12
- J1 pad 13: c1 -> ch13
- J1 pad 14: c0 -> ch14
- J1 pad 15: ec1b -> ch15
- J1 pad 16: ec1a -> ch16
- J1 pad 17: gpio3 -> ch17
- J1 pad 18: row_d -> ch18
- J1 pad 19: row_c -> ch19
- J1 pad 2: row_h -> ch2
- J1 pad 20: row_b -> ch20
- J1 pad 21: row_a -> ch21
- J1 pad 3: row_g -> ch3
- J1 pad 4: row_f -> ch4
- J1 pad 6: gpio4 -> ch6
- J1 pad 7: ec2b -> ch7
- J1 pad 8: ec2a -> ch8
- J1 pad 9: c5 -> ch9
- J3 pad 1: VCC -> VDD
- J4 pad A1: GND -> Net-(FB5-Pad2)
- J4 pad A12: GND -> Net-(FB5-Pad2)
- J4 pad A4: Net-(FB1-Pad1) -> Net-(C4--)
- J4 pad A6: /power/IN_D+ -> D+
- J4 pad A7: /power/IN_D- -> D-
- J4 pad A9: Net-(FB1-Pad1) -> Net-(C4--)
- J4 pad B1: GND -> Net-(FB5-Pad2)
- J4 pad B12: GND -> Net-(FB5-Pad2)
- J4 pad B4: Net-(FB1-Pad1) -> Net-(C4--)
- J4 pad B6: /power/IN_D+ -> D+
- J4 pad B7: /power/IN_D- -> D-
- J4 pad B9: Net-(FB1-Pad1) -> Net-(C4--)
- J5 pad 1: Net-(D4-K) -> Net-(J5-Pin_1)
- J6 pad 1: mosi -> sck
- J6 pad 2: sck -> mosi
- J6 pad 3: VCC -> cs
- J6 pad 4: GND -> Net-(J6-Pin_4)
- J6 pad 5: cs -> Net-(J6-Pin_5)
- JP1 pad 1: VCC -> PRI_MID
- JP1 pad 2: Net-(D4-K) -> Net-(J5-Pin_1)
- R2 pad 2: Net-(JP4-B) -> status_led_1
- R7 pad 2: status_led -> status_led_2
- SW1 pad 2: Net-(U1-P0.30) -> Net-(U1-P1.03)
- U1 pad 10: sda -> ch21
- U1 pad 14: VCC -> VDC
- U1 pad 16: VCC -> VDD
- U1 pad 17: unconnected-(U1-P0.13-Pad17) -> ch13
- U1 pad 18: c0 -> ch12
- U1 pad 19: c1 -> ch11
- U1 pad 20: c2 -> ch10
- U1 pad 21: c3 -> ch9
- U1 pad 22: c4 -> ch8
- U1 pad 23: c5 -> ch7
- U1 pad 24: unconnected-(U1-P1.07-Pad24) -> ch2
- U1 pad 25: gpio4 -> ch3
- U1 pad 26: BATT_READ -> ch4
- U1 pad 28: row_f -> ch6
- U1 pad 29: row_g -> unconnected-(U1-P0.21-Pad29)
- U1 pad 3: scl -> Net-(U1-P1.03)
- U1 pad 30: row_h -> unconnected-(U1-P1.06-Pad30)
- U1 pad 31: unconnected-(U1-P0.27-Pad31) -> BATT_READ_EN
- U1 pad 33: ec2a -> BATT_READ
- U1 pad 34: ec2b -> led_data
- U1 pad 37: Net-(U1-P0.30) -> ch14
- U1 pad 38: led_data -> ch15
- U1 pad 39: unconnected-(U1-P1.11-Pad39) -> ch16
- U1 pad 4: ec1b -> status_led_2
- U1 pad 40: gpio3 -> ch17
- U1 pad 41: gpio1 -> ch18
- U1 pad 42: gpio2 -> ch19
- U1 pad 43: unconnected-(U1-P1.15-Pad43) -> ch20
- U1 pad 47: status_led -> unconnected-(U1-P0.03-Pad47)
- U1 pad 5: ec1a -> status_led_1
- U1 pad 58: BATT_READ_EN -> unconnected-(U1-P0.26-Pad58)
- U1 pad 6: row_d -> scl
- U1 pad 7: row_c -> sda
- U1 pad 8: row_b -> gpio1
- U1 pad 9: row_a -> gpio2
- U2 pad 1: Net-(D45-K) -> VDC
- U2 pad 3: Net-(D45-K) -> VDC
Routing:
- net VCC: track 181.6 -> 48.2 mm, vias 9 -> 0
- net status_led_2: track 0.00 -> 126.3 mm, vias 0 -> 2
- net status_led_1: track 0.00 -> 99.5 mm, vias 0 -> 2
- net /power/IN_D+: track 87.6 -> 0.00 mm, vias 4 -> 0
- net /power/IN_D-: track 87.2 -> 0.00 mm, vias 2 -> 0
- net D-: track 6.36 -> 88.0 mm
- net D+: track 7.90 -> 86.9 mm, vias 2 -> 4
- net VDC: track 0.00 -> 76.3 mm, vias 0 -> 2
- net Net-(D45-K): track 51.0 -> 0.00 mm, vias 2 -> 0
- net Net-(U1-P1.03): track 0.00 -> 45.9 mm, vias 0 -> 1
- net Net-(U1-P0.30): track 41.7 -> 0.00 mm, vias 3 -> 0
- net sck: track 17.6 -> 56.0 mm, vias 3 -> 2
- net status_led: track 32.4 -> 0.00 mm, vias 4 -> 0
- net ec2b: track 29.9 -> 0.00 mm, vias 2 -> 0
- net ch14: track 0.00 -> 29.2 mm, vias 0 -> 2
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Other:
- board size 52.1 x 109 mm -> 49.4 x 106.4 mm
- board text added: "+"
- board text added: "10nF"
- board text added: "2"
- board text added: "2k"
- board text added: "3"
- board text added: "3.3v reg"
- board text added: "battery pwr"
- board text added: "reset"
- board text added: "sao pwr"
- board text added: "swdclk"
- board text added: "swdio"
- board text removed: "22"
- board text removed: "3k"
- board text removed: "VCC reg"
- board text removed: "bat pwr"
- board text removed: "by"
- board text removed: "sao power"
- board text removed: "status"
- board text removed: "vbus"
- board text removed: "vcc"

Commit message: mariposa v2 RC3
Parts:
- removed D2, D3, D4: D_Schottky, PCM_Diode_SMD_Handsoldering_AKL:D_SOD-123F
- removed J5: Conn_02x03_Counter_Clockwise, Connector_PinSocket_2.54mm:PinSocket_2x03_P2.54mm_Vertical_SMD
- removed JP1: SolderJumper_2_Open, Jumper:SolderJumper-2_P1.3mm_Open_TrianglePad1.0x1.5mm
- removed R1: 20k, Resistor_SMD:R_0603_1608Metric
- removed SW2: Slide_DPDT_SS22D06, Button_Switch_SMD:SW_DPDT_CK_JS202011JCQN
- removed TP5: TestPoint, TestPoint:TestPoint_Pad_D1.0mm
- removed U3: MCP73831T-2ACI/OT, Package_TO_SOT_SMD:SOT-23-5
- added J8: Conn_01x04_MountingPin, Connector_JST:JST_SH_SM04B-SRSS-TB_1x04-1MP_P1.00mm_Horizontal, B.Cu at (136.1, 52.3)
- added J9: Conn_02x03_Odd_Even, Connector_PinSocket_2.54mm:PinSocket_2x03_P2.54mm_Vertical_SMD, F.Cu at (140.1, 52.5)
- added L1: 1 uH, Inductor_SMD:L_0603_1608Metric, B.Cu at (164.2, 74.5)
- added R11: 249k, Resistor_SMD:R_0603_1608Metric, B.Cu at (162.7, 69.8)
- added R12: 10k, Resistor_SMD:R_0603_1608Metric, B.Cu at (165.7, 50.6)
- added R14: 10k, Resistor_SMD:R_0603_1608Metric, B.Cu at (167.1, 40.3)
- added R15: 27k, Resistor_SMD:R_0603_1608Metric, B.Cu at (167.9, 54.1)
- added U4: TPS22917DBV, Package_TO_SOT_SMD:SOT-23-6, B.Cu at (144.0, 60.6)
- added U5: TPS628438DRL, Package_TO_SOT_SMD:SOT-563, B.Cu at (164.9, 72.5)
- C4, C5: footprint Capacitor_SMD:C_0402_1005Metric -> Capacitor_SMD:C_0603_1608Metric
- C44: value 1uF -> 4.7 uF
- C45: value 1uF -> 10 uF
- C46, C47: value 4.7uF -> 1uF
- D1: footprint PCM_LED_SMD_AKL:LED_1206_3216Metric_ReverseMount_Hole1.8x2.4mm -> coquette_footprints:LED 1206 reverse mount rectangle
- D5, D6: footprint LED_SMD:LED_1206_3216Metric_ReverseMount_Hole1.8x2.4mm -> coquette_footprints:LED 1206 reverse mount rectangle
- FB6, FB7: value 240 Ohm -> 120 Ohm
- R2, R7: value 2k -> 1.5k
- R9: value 800K -> 800k
- U2: value TPS7A0333PDBVR -> BQ25170DSGR; footprint Package_TO_SOT_SMD:SOT-23-5 -> coquette_footprints:DSG0008A
- moved R8 22.8 mm to (153.2, 73.8), turned to 180 degrees
- moved D45 16.8 mm to (169.3, 66.9), turned to 90 degrees
- moved C44 15.2 mm to (167.4, 72.3)
- moved TP4 14.1 mm to (156.2, 94.9)
- moved U2 11.9 mm to (164.5, 54.0)
- moved FB6 10.8 mm to (141.6, 66.1)
- moved R7 10.7 mm to (164.1, 50.6), turned to 90 degrees
- moved D88 9.49 mm to (159.4, 66.9)
- moved C45 8.20 mm to (163.1, 72.2), turned to 90 degrees
- moved C46 7.64 mm to (162.4, 52.3), turned to -90 degrees
- moved C47 2.89 mm to (161.6, 55.2)
- moved J2 2.56 mm to (133.9, 59.6)
- moved BT1 2.49 mm to (166.7, 59.2)
- moved C4 2.49 mm to (157.0, 52.1)
- moved C5 2.33 mm to (157.0, 56.9)
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Connections:
- D10 pad 1: gpio1 -> D-
- D10 pad 3: D- -> gpio1
- D10 pad 4: D+ -> gpio2
- D10 pad 6: gpio2 -> D+
- D11 pad 1: VCC -> unconnected-(D11-L1-Pad1)
- D12 pad 1: status_led_2 -> led_data
- D13 pad 1: VDD -> VCC
- D45 pad 2: +3V8 -> +BATT
- D5 pad 1: GND -> status_led_1
- D6 pad 1: GND -> Net-(D6-K)
- FB6 pad 2: Net-(D4-K) -> VCC
- J2 pad 2: +5V -> PRI_LO
- J2 pad 3: GND -> Earth_Clean
- J3 pad 1: VDD -> VCC
- J7 pad 2: Earth_Clean -> GND
- R2 pad 2: status_led_1 -> VCC
- R7 pad 1: Net-(D6-A) -> Net-(U2-ISET)
- R7 pad 2: status_led_2 -> GND
- R8 pad 1: Net-(U3-PROG) -> VBUS
- R8 pad 2: GND -> Net-(D1-A)
- R9 pad 1: +3V8 -> +BATT
- U1 pad 14: VDC -> VCC
- U1 pad 16: VDD -> VCC
- U1 pad 34: led_data -> unconnected-(U1-P1.10-Pad34)
- U1 pad 4: status_led_2 -> scl
- U1 pad 49: unconnected-(U1-P0.22-Pad49) -> ext_on
- U1 pad 5: status_led_1 -> sda
- U1 pad 6: scl -> gpio2
- U1 pad 7: sda -> gpio1
- U1 pad 8: gpio1 -> status_led_1
- U1 pad 9: gpio2 -> led_data
- U2 pad 1: VDC -> VBUS
- U2 pad 2: GND -> Net-(U2-ISET)
- U2 pad 3: VDC -> Net-(U2-TS)
- U2 pad 4: unconnected-(U2-NC-Pad4) -> GND
- U2 pad 5: VCC -> Net-(D1-K)
Routing:
- net VCC: track 48.2 -> 198.0 mm, vias 0 -> 6
- net status_led_2: track 126.3 -> 0.00 mm, vias 2 -> 0
- net +3V8: track 105.5 -> 0.00 mm, vias 2 -> 0
- net +BATT: track 18.9 -> 92.5 mm
- net ext_on: track 0.00 -> 72.7 mm, vias 0 -> 4
- net VBUS: track 88.3 -> 119.9 mm, vias 2 -> 0
- net VDC: track 76.3 -> 46.1 mm, vias 2 -> 4
- net Net-(D6-K): track 0.00 -> 27.6 mm, vias 0 -> 2
- net Earth_Clean: track 8.96 -> 31.1 mm, vias 0 -> 1
- net Net-(D4-K): track 22.0 -> 0.00 mm, vias 2 -> 0
- net VDD: track 18.3 -> 0.00 mm, vias 1 -> 0
- net +5V: track 17.0 -> 0.00 mm
- net PRI_LO: track 0.00 -> 10.9 mm
- net led_data: track 98.2 -> 88.2 mm
- net scl: track 83.0 -> 90.7 mm
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- added copper zone on B.Cu, net +BATT
- added copper zone on B.Cu, net Earth_Clean
- added copper zone on B.Cu, net VBUS
- added copper zone on B.Cu, net VCC
- added copper zone on B.Cu, net VDC
Other:
- board text added: "1.5k"
- board text added: "10uF"
- board text added: "1uH"
- board text added: "249k"
- board text added: "27k"
- board text added: "3V reg"
- board text added: "560pF"
- board text added: "cs"
- board text added: "cutie"
- board text added: "debug"
- board text added: "fb 240"
- board text added: "mosi"
- board text added: "power"
- board text added: "rgb out"
- board text added: "rgb switch"
- board text added: "sck"
- board text added: "status"
- board text added: "vcc"
- board text removed: "2"
- board text removed: "20k"
- board text removed: "2k"
- board text removed: "3"
- board text removed: "3.3v reg"
- board text removed: "bat"
- board text removed: "battery pwr"
- board text removed: "rgb"
- board text removed: "sao pwr"

Commit message: parpar mariposa mk2 rc6
Routing:
- net Net-(D6-K): track 27.6 -> 28.2 mm
Other:
- board text added: "3V3 reg"
- board text removed: "3V reg"
