File: mariposa.kicad_pcb (KiCad board)
At the start: 6 copper layers, 36 x 77.5 mm, 88 parts, among them J1 Conn_01x28_MountingPin, J2 Conn_01x03_MountingPin, J3 Conn_ARM_SWD_TagConnect_TC203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, J4 USB_C_Receptacle_USB2.0_16P, J5 Conn_01x08_MountingPin, J6 Conn_01x10_MountingPin, J8 Conn_01x04_MountingPin, J9 Conn_02x03_Odd_Even, SW1 SW_Push, SW3 SW_Push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

Commit message: new dcdc rerouting
Routing:
- net GND: track 38.0 -> 51.6 mm, vias 195 -> 190
- net vcc_mode: track 0.00 -> 7.59 mm, vias 1 -> 2
- net ll_oe: track 14.8 -> 21.3 mm
- net +BATT: track 63.1 -> 65.2 mm
- net argb: track 52.8 -> 53.8 mm
- net VCC: vias 28 -> 29
Other:
- board text added: "vset"
- board text removed: "0.1"
- board text removed: "52.3k"

Commit message: tweaks
Parts:
- C44, C48, C49: footprint Capacitor_SMD:C_0603_1608Metric -> Capacitor_SMD:C_1206_3216Metric
- C45, C53: footprint Capacitor_SMD:C_0603_1608Metric -> Capacitor_SMD:C_0805_2012Metric
- R21: footprint Resistor_SMD:R_0603_1608Metric -> Resistor_SMD:R_0805_2012Metric
- moved C44 9.22 mm to (140.2, 96.0), turned to 0 degrees
- moved C45 7.65 mm to (131.2, 100.5), turned to 90 degrees
- moved C48 2.85 mm to (140.0, 115.1), turned to -90 degrees
- moved R21 2.57 mm to (139.8, 119.2)
- moved C49 1.84 mm to (143.1, 115.1)
- moved R11 1.58 mm to (135.5, 107.7), turned to -90 degrees
- moved C53 0.33 mm to (153.5, 66.8)
Routing:
- net GND: track 51.6 -> 66.3 mm, vias 190 -> 185
- net VDC: track 72.1 -> 65.2 mm
- net VCC: track 39.1 -> 44.3 mm, vias 29 -> 28
- net PRI_LO: track 39.1 -> 42.6 mm
- net VBUS: track 110.4 -> 107.1 mm, vias 9 -> 8
- net Net-(U1-VSET): track 5.41 -> 2.57 mm
- net vcc_mode: track 7.59 -> 8.86 mm
- net Net-(MDBT1-VBUS): track 4.77 -> 3.65 mm
- net Net-(JP2-A): track 8.15 -> 7.64 mm
