File: mariposa.kicad_sch (KiCad schematic)
At the start: 41 parts, among them J1 Conn_01x28_MountingPin, J3 Conn_ARM_SWD_TagConnect_TC203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, J6 Conn_01x10_MountingPin, J8 Conn_01x04_MountingPin, J9 Conn_02x03_Odd_Even, SW1 SW_Push, SW3 SW_Push

Commit message: title page 3 of schematic
Other:
- moved on the sheet: TP1, TP2, TP3, TP4, TP6, TP7, TP8
Changed lines of the file:
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@@
 	)
 	(rectangle
-		(start 129.54 110.49)
-		(end 189.865 140.97)
+		(start 124.46 115.57)
+		(end 184.785 146.05)
 		(stroke
 			(width 0)
@@
 	(text "test points"
 		(exclude_from_sim no)
-		(at 134.874 109.474 0)
+		(at 129.794 114.554 0)
 		(effects
 			(font
@@
 	(global_label "sck"
 		(shape input)
-		(at 139.7 133.35 270)
+		(at 134.62 138.43 270)
 		(fields_autoplaced yes)
 		(effects
@@
 		)
 		(property "Intersheetrefs" "${INTERSHEET_REFS}"
-			(at 139.7 138.8709 90)
+			(at 134.62 143.9509 90)
 			(effects
 				(font
@@
 	(global_label "swdio"
 		(shape input)
-		(at 148.59 118.11 270)
+		(at 143.51 123.19 270)
 		(fields_autoplaced yes)
 		(effects
@@
 		)
 		(property "Intersheetrefs" "${INTERSHEET_REFS}"
-			(at 148.59 125.4697 90)
+			(at 143.51 130.5497 90)
 			(effects
 				(font
@@
 	(global_label "reset"
 		(shape input)
-		(at 162.56 118.11 270)
+		(at 157.48 123.19 270)
 		(fields_autoplaced yes)
 		(effects
@@
 		)
 		(property "Intersheetrefs" "${INTERSHEET_REFS}"
-			(at 162.56 125.4697 90)
+			(at 157.48 130.5497 90)
 			(effects
 				(font
@@
 	(global_label "cs"
 		(shape input)
-		(at 167.64 133.35 270)
+		(at 162.56 138.43 270)
 		(fields_autoplaced yes)
 		(effects
@@
 		)
 		(property "Intersheetrefs" "${INTERSHEET_REFS}"
-			(at 167.64 137.9515 90)
+			(at 162.56 143.0315 90)
 			(effects
 				(font
@@
 	(global_label "swdclk"
 		(shape input)
-		(at 134.62 118.11 270)
+		(at 129.54 123.19 270)
 		(fields_autoplaced yes)
 		(effects
@@
 		)
 		(property "Intersheetrefs" "${INTERSHEET_REFS}"
-			(at 134.62 126.3891 90)
+			(at 129.54 131.4691 90)
 			(effects
 				(font
@@
 	(global_label "mosi"
 		(shape input)
-		(at 153.67 133.35 270)
+		(at 148.59 138.43 270)
 		(fields_autoplaced yes)
 		(effects
@@
 		)
 		(property "Intersheetrefs" "${INTERSHEET_REFS}"
-			(at 153.67 139.7903 90)
+			(at 148.59 144.8703 90)
 			(effects
 				(font
@@
 	(symbol
 		(lib_id "Connector:TestPoint")
-		(at 148.59 118.11 0)
+		(at 143.51 123.19 0)
 		(unit 1)
 		(exclude_from_sim no)
@@
 		(fields_autoplaced yes)
 		(property "Reference" "TP2"
-			(at 151.13 113.5379 0)
+			(at 146.05 118.6179 0)
 			(effects
 				(font
@@
 		)
 		(property "Value" "TestPoint"
-			(at 151.13 116.0779 0)
+			(at 146.05 121.1579 0)
 			(effects
 				(font
@@
 		)
 		(property "Footprint" "TestPoint:TestPoint_Pad_D1.0mm"
-			(at 153.67 118.11 0)
+			(at 148.59 123.19 0)
 			(effects
 				(font
@@
 		)
 		(property "Datasheet" "~"
-			(at 153.67 118.11 0)
+			(at 148.59 123.19 0)
 			(effects
 				(font
@@
 		)
 		(property "Description" "test point"
-			(at 148.59 118.11 0)
+			(at 143.51 123.19 0)
 			(effects
 				(font
@@
 	(symbol
 		(lib_id "power:VCC")
-		(at 176.53 118.11 180)
+		(at 171.45 123.19 180)
 		(unit 1)
 		(exclude_from_sim no)
@@
 		(dnp no)
 		(property "Reference" "#PWR040"
-			(at 176.53 114.3 0)
+			(at 171.45 119.38 0)
 			(effects
 				(font
@@
 		)
 		(property "Value" "VCC"
-			(at 176.53 123.19 90)
+			(at 171.45 128.27 90)
 			(effects
 				(font
@@
 		)
 		(property "Footprint" ""
-			(at 176.53 118.11 0)
+			(at 171.45 123.19 0)
 			(effects
 				(font
@@
 		)
 		(property "Datasheet" ""
-			(at 176.53 118.11 0)
+			(at 171.45 123.19 0)
 			(effects
 				(font
@@
 		)
 		(property "Description" "Power symbol creates a global label with name \"VCC\""
-			(at 176.53 118.11 0)
+			(at 171.45 123.19 0)
 			(effects
 				(font
@@
 	(symbol
 		(lib_id "Connector:TestPoint")
-		(at 162.56 118.11 0)
+		(at 157.48 123.19 0)
 		(unit 1)
 		(exclude_from_sim no)
@@
 		(fields_autoplaced yes)
 		(property "Reference" "TP3"
-			(at 165.1 113.5379 0)
+			(at 160.02 118.6179 0)
 			(effects
 				(font
@@
 		)
 		(property "Value" "TestPoint"
-			(at 165.1 116.0779 0)
+			(at 160.02 121.1579 0)
 			(effects
 				(font
@@
 		)
 		(property "Footprint" "TestPoint:TestPoint_Pad_D1.0mm"
-			(at 167.64 118.11 0)
+			(at 162.56 123.19 0)
 			(effects
 				(font
@@
 		)
 		(property "Datasheet" "~"
-			(at 167.64 118.11 0)
+			(at 162.56 123.19 0)
 			(effects
 				(font
@@
 		)
 		(property "Description" "test point"
-			(at 162.56 118.11 0)
+			(at 157.48 123.19 0)
 			(effects
 				(font
@@
 	(symbol
 		(lib_id "Connector:TestPoint")
-		(at 139.7 133.35 0)
+		(at 134.62 138.43 0)
 		(unit 1)
 		(exclude_from_sim no)
@@
 		(fields_autoplaced yes)
 		(property "Reference" "TP6"
-			(at 142.24 128.7779 0)
+			(at 137.16 133.8579 0)
 			(effects
 				(font
@@
 		)
 		(property "Value" "TestPoint"
-			(at 142.24 131.3179 0)
+			(at 137.16 136.3979 0)
 			(effects
 				(font
@@
 		)
 		(property "Footprint" "TestPoint:TestPoint_Pad_D1.0mm"
-			(at 144.78 133.35 0)
+			(at 139.7 138.43 0)
 			(effects
 				(font
@@
 		)
 		(property "Datasheet" "~"
-			(at 144.78 133.35 0)
+			(at 139.7 138.43 0)
 			(effects
 				(font
@@
 		)
 		(property "Description" "test point"
-			(at 139.7 133.35 0)
+			(at 134.62 138.43 0)
 			(effects
 				(font
@@
 	(symbol
 		(lib_id "Connector:TestPoint")
-		(at 176.53 118.11 0)
+		(at 171.45 123.19 0)
 		(unit 1)
 		(exclude_from_sim no)
@@
 		(fields_autoplaced yes)
 		(property "Reference" "TP4"
-			(at 179.07 113.5379 0)
+			(at 173.99 118.6179 0)
 			(effects
 				(font
@@
 		)
 		(property "Value" "TestPoint"
-			(at 179.07 116.0779 0)
+			(at 173.99 121.1579 0)
 			(effects
 				(font
@@
 		)
 		(property "Footprint" "TestPoint:TestPoint_Pad_D1.0mm"
-			(at 181.61 118.11 0)
+			(at 176.53 123.19 0)
 			(effects
 				(font
@@
 		)
 		(property "Datasheet" "~"
-			(at 181.61 118.11 0)
+			(at 176.53 123.19 0)
 			(effects
 				(font
@@
 		)
 		(property "Description" "test point"
-			(at 176.53 118.11 0)
+			(at 171.45 123.19 0)
 			(effects
 				(font
@@
 	(symbol
 		(lib_id "Connector:TestPoint")
-		(at 134.62 118.11 0)
+		(at 129.54 123.19 0)
 		(unit 1)
 		(exclude_from_sim no)
@@
 		(fields_autoplaced yes)
 		(property "Reference" "TP1"
-			(at 137.16 113.5379 0)
+			(at 132.08 118.6179 0)
 			(effects
 				(font
@@
 		)
 		(property "Value" "TestPoint"
-			(at 137.16 116.0779 0)
+			(at 132.08 121.1579 0)
 			(effects
 				(font
@@
 		)
 		(property "Footprint" "TestPoint:TestPoint_Pad_D1.0mm"
-			(at 139.7 118.11 0)
+			(at 134.62 123.19 0)
 			(effects
 				(font
@@
 		)
 		(property "Datasheet" "~"
-			(at 139.7 118.11 0)
+			(at 134.62 123.19 0)
 			(effects
 				(font
@@
 		)
 		(property "Description" "test point"
-			(at 134.62 118.11 0)
+			(at 129.54 123.19 0)
 			(effects
 				(font
@@
 	(symbol
 		(lib_id "Connector:TestPoint")
-		(at 167.64 133.35 0)
+		(at 162.56 138.43 0)
 		(unit 1)
 		(exclude_from_sim no)
@@
 		(fields_autoplaced yes)
 		(property "Reference" "TP8"
-			(at 170.18 128.7779 0)
+			(at 165.1 133.8579 0)
 			(effects
 				(font
@@
 		)
 		(property "Value" "TestPoint"
-			(at 170.18 131.3179 0)
+			(at 165.1 136.3979 0)
 			(effects
 				(font
@@
 		)
 		(property "Footprint" "TestPoint:TestPoint_Pad_D1.0mm"
-			(at 172.72 133.35 0)
+			(at 167.64 138.43 0)
 			(effects
 				(font
@@
 		)
 		(property "Datasheet" "~"
-			(at 172.72 133.35 0)
+			(at 167.64 138.43 0)
 			(effects
 				(font
@@
 		)
 		(property "Description" "test point"
-			(at 167.64 133.35 0)
+			(at 162.56 138.43 0)
 			(effects
 				(font
@@
 	(symbol
 		(lib_id "Connector:TestPoint")
-		(at 153.67 133.35 0)
+		(at 148.59 138.43 0)
 		(unit 1)
 		(exclude_from_sim no)
@@
 		(fields_autoplaced yes)
 		(property "Reference" "TP7"
-			(at 156.21 128.7779 0)
+			(at 151.13 133.8579 0)
 			(effects
 				(font
@@
 		)
 		(property "Value" "TestPoint"
-			(at 156.21 131.3179 0)
+			(at 151.13 136.3979 0)
 			(effects
 				(font
@@
 		)
 		(property "Footprint" "TestPoint:TestPoint_Pad_D1.0mm"
-			(at 158.75 133.35 0)
+			(at 153.67 138.43 0)
 			(effects
 				(font
@@
 		)
 		(property "Datasheet" "~"
-			(at 158.75 133.35 0)
+			(at 153.67 138.43 0)
 			(effects
 				(font
@@
 		)
 		(property "Description" "test point"
-			(at 153.67 133.35 0)
+			(at 148.59 138.43 0)
 			(effects
 				(font

Commit message: cleanup
Parts:
- added RN4: 2*10k, PCM_Resistor_SMD_AKL:R_Array_Convex_2x0402, symbol PCM_Resistor_US_AKL:R_2x0402_Convex
- TP1, TP2, TP3, TP4: now left out of the parts list
Connections:
- net VCC: now also RN4.1 (R1.1), RN4.2 (R2.1)
- net scl: now also RN4.4 (R1.2)
- net sda: now also RN4.3 (R2.2)
Other:
- note added: "i2c pull-up"
- note added: "internal pull-up override"
- moved on the sheet: H2, H3, H4, H5

Commit message: v3 efforts
Parts:
- removed C10: 1uF, Capacitor_SMD:C_0603_1608Metric, symbol Device:C
- removed C12: 10nF, Capacitor_SMD:C_0402_1005Metric, symbol PCM_Elektuur:C
- removed FB5: 120 Ohm, PCM_Ferrite_SMD_AKL:Ferrite_0805_2012Metric, symbol PCM_Device_AKL:Ferrite_Bead
- removed J8: Conn_01x04_MountingPin, Connector_JST:JST_SH_SM04B-SRSS-TB_1x04-1MP_P1.00mm_Horizontal, symbol Connector_Generic_MountingPin:Conn_01x04_MountingPin
- removed J9: Conn_02x03_Odd_Even, Connector_PinSocket_2.54mm:PinSocket_2x03_P2.54mm_Vertical_SMD, symbol Connector_Generic:Conn_02x03_Odd_Even
- removed JP1: SolderJumper_3_Bridged12, Jumper:SolderJumper-3_P1.3mm_Bridged12_RoundedPad1.0x1.5mm, symbol Jumper:SolderJumper_3_Bridged12
- removed R1, R16: R220, Resistor_SMD:R_0603_1608Metric, symbol Device:R_US
- removed R13: 10k, Resistor_SMD:R_0603_1608Metric, symbol Device:R_US
- removed R17: R2.2, Resistor_SMD:R_0603_1608Metric, symbol Device:R_US
- removed R19, R20: 1.67k, Resistor_SMD:R_0402_1005Metric, symbol Device:R_US
- removed R2: 5k, Resistor_SMD:R_0402_1005Metric, symbol Device:R_US
- removed RN3: 2*R33, PCM_Resistor_SMD_AKL:R_Array_Convex_2x0402, symbol PCM_Resistor_US_AKL:R_2x0402_Convex
- removed RN4: 2*10k, PCM_Resistor_SMD_AKL:R_Array_Convex_2x0402, symbol PCM_Resistor_US_AKL:R_2x0402_Convex
- removed TP1, TP2, TP3, TP6, TP7, TP8: TestPoint, TestPoint:TestPoint_Pad_D1.0mm, symbol Connector:TestPoint
- removed U1: ~, coquette_footprints:holyiot_21069_nRF5340, symbol coquette_symbols:holyiot_21069_nrf5340
- added C18, C19: 1uF, Capacitor_SMD:C_0603_1608Metric, symbol Device:C
- added C48, C49: 4.7uF, Capacitor_SMD:C_0603_1608Metric, symbol Device:C
- added L2, L3: 10uH, Inductor_SMD:L_0603_1608Metric, symbol PCM_Generic-50:L,IEEE
- added MDBT1: ~, coquette_footprints:MDBT53, symbol coquette_symbols:MDBT53
- added R21: R2.2, Resistor_SMD:R_0603_1608Metric, symbol Device:R_US
- added RN5: 2*R27, Resistor_SMD:R_Array_Convex_2x0603, symbol PCM_Resistor_US_AKL:R_2x0402_Convex
- added RN6, RN7: 10k*4, PCM_Resistor_SMD_AKL:R_Array_Convex_4x0603, symbol PCM_Resistor_US_AKL:R_4x0603_Convex
- added TP5: TestPoint, TestPoint:TestPoint_Pad_D1.0mm, symbol Connector:TestPoint
- added Y1: CFPX-217 32.768KHz, Crystal:Crystal_SMD_3215-2Pin_3.2x1.5mm, symbol Device:Crystal
- J1: footprint coquette_footprints:AMPHENOL_SFV28R-1STE1HLF -> Connector_FFC-FPC:Hirose_FH12-28S-0.5SH_1x28-1MP_P0.50mm_Horizontal
- J6: footprint coquette_footprints:AMPHENOL_SFV10R-1STE1HLF -> Connector_FFC-FPC:Hirose_FH12-10S-0.5SH_1x10-1MP_P0.50mm_Horizontal
- R5, R6: value 10k -> 1.5k
- RN1, RN2: footprint PCM_Resistor_SMD_AKL:R_Array_Convex_2x0402 -> Resistor_SMD:R_Array_Convex_2x0603
- SW1, SW3: footprint Button_Switch_SMD:SW_SPST_PTS645 -> coquette_footprints:G-Switch GT-TC041B-H036-L1N
Connections:
- net gpio1 is gone; now on net sda: RN2.4 (R1.2)
- net BATT_READ: now also MDBT1.60 (P0.28/AIN7)
- net BATT_READ_EN: now also MDBT1.59 (P1.10)
- net D+: now also RN5.1 (R1.1)
- net D-: now also RN5.2 (R2.1)
- net GND: now also SW1.2, C18.1, C19.1, C48.1, C49.1, MDBT1.1 (GND@1), MDBT1.24 (GND@24), MDBT1.42 (GND@42), MDBT1.61 (GND@61), RN7.7 (R2.2), RN7.8 (R1.2); no longer R5.1, SW1.1
- net VBUS: now also C48.2, R21.2
- net VCC: now also C49.2, MDBT1.38 (VDD), MDBT1.41 (VDDH), RN7.6 (R3.2); no longer R6.2
- net argb: now also MDBT1.65 (P0.29)
- net ch1: now also MDBT1.56 (P0.31)
- net ch10: now also MDBT1.27 (P0.14/QSPI1)
- net ch11: now also MDBT1.26 (P0.17/QSPI_SCK)
- net ch12: now also MDBT1.23 (P0.15/QSPI2)
- net ch13: now also MDBT1.25 (P0.22)
- net ch14: now also MDBT1.22 (P1.05)
- net ch15: now also MDBT1.21 (P0.13/QSPI0)
- net ch16: now also MDBT1.20 (P0.07/AIN3)
- net ch17: now also MDBT1.9 (P0.25/AIN4)
- net ch18: now also MDBT1.7 (P0.26/AIN5)
- net ch19: now also MDBT1.16 (P0.18/QSPI_CSN)
- net ch2: now also MDBT1.55 (P1.11)
- net ch20: now also MDBT1.14 (P0.19)
- net ch21: now also MDBT1.13 (P0.20)
- net ch22: now also MDBT1.12 (P0.21)
- net ch23: now also MDBT1.11 (P1.04)
- net ch24: now also MDBT1.10 (P1.06)
- net ch3: now also MDBT1.51 (P1.13)
- net ch4: now also MDBT1.49 (P1.14)
- net ch5: now also MDBT1.45 (P1.00)
- net ch6: now also MDBT1.43 (P1.01)
- net ch7: now also MDBT1.47 (P1.15)
- net ch8: now also MDBT1.53 (P1.12)
- net ch9: now also MDBT1.28 (P0.16/QSPI3)
- net chg_stat: now also MDBT1.8 (P0.24)
- net cs: now also MDBT1.17 (P0.11/HSPI_CSN)
- net eepy: now also R5.1, MDBT1.57 (P0.30); no longer SW1.2
- net ext_on: now also MDBT1.5 (P0.27/AIN6)
- net gpio2: now also MDBT1.35 (P0.06/AIN2); no longer RN2.3 (R2.2)
- net miso: now also MDBT1.18 (P0.10/HSPI_MISO)
- net mosi: now also MDBT1.19 (P0.09/HSPI_MOSI)
- net reset: now also R6.1, MDBT1.6 (RESET); no longer SW3.1
- net sck: now also MDBT1.29 (P0.08/HSPI_SCK)
- net scl: now also RN2.3 (R2.2)
- net swdclk: now also RN1.3 (R2.2); no longer RN1.4 (R1.2)
- net swdio: now also RN1.4 (R1.2); no longer RN1.3 (R2.2)
- net stat_red: now reaches LED1.1 (R)
- net stat_red: now also RN6.3 (R3.1)
- net disp: now reaches C1.1, J6.5 (Pin_5)
- net disp: now also RN7.3 (R3.1); no longer R6.1
- net at R5.2: now also SW3.1; no longer J6.4 (Pin_4)
- net at RN2.1 (R1.1): now also MDBT1.33 (P1.02/TWI)
- net at RN2.2 (R2.1): now also MDBT1.31 (P1.03/TWI)
- net at RN1.1 (R1.1): now also MDBT1.4 (SWDIO)
- net at RN1.2 (R2.1): now also MDBT1.2 (SWDCLK)
- net stat_green: now reaches LED1.3 (G)
- net stat_green: now also RN6.4 (R4.1)
- net stat_blue: now reaches LED1.4 (B)
- net stat_blue: now also RN6.2 (R2.1)
- net extmode: now reaches J6.8 (Pin_8)
- net extmode: now also RN7.1 (R1.1)
- new net: C18.2, L2.1 (+), MDBT1.52 (DECD)
- new net: L2.2 (-), MDBT1.50 (DCCD)
- new net: R6.2, SW1.1
- new net: MDBT1.36 (P0.01/XL2), Y1.1
- new net: MDBT1.34 (P0.00/XL1), Y1.2
- new net: L3.1 (+), MDBT1.54 (DCC)
- new net: C19.2, L3.2 (-), MDBT1.58 (DECR)
- new net: MDBT1.44 (VBUS), R21.1
- new net MCU_D+: MDBT1.46 (D+), RN5.4 (R1.2)
- new net MCU_D-: MDBT1.48 (D-), RN5.3 (R2.2)
- new net VDC: RN6.1 (R1.1)
- new net argb_data: TP5.1
- new net chg_pg: MDBT1.3 (P1.08)
- new net dcx: MDBT1.15 (P0.12/HSPI_DCX)
- new net extcomin: J6.4 (Pin_4), RN7.2 (R2.1)
- new net ll_oe: RN7.4 (R4.1)
- new net ll_pull_down: RN7.5 (R4.2)
- new net status_led_blue: MDBT1.62 (P0.23), RN6.5 (R4.2)
- new net status_led_green: MDBT1.63 (P1.07), RN6.6 (R3.2)
- new net status_led_red: MDBT1.64 (P1.09), RN6.7 (R2.2)
- new net vcc_en: RN6.8 (R1.2)
- no-connect marks 8 -> 5
Other:
- added sheet addons (addons.kicad_sch)
- note removed: "i2c pull-up"
- note removed: "internal pull-up override"
- note removed: "microcontroller and debug header"
- note removed: "sao v1.69bis"
- note removed: "stemma qt"
- moved on the sheet: C1, C2, C3, FB3, FB4, H2, H3, H4, H5, J1, J3, J6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

Commit message: more rounding
Connections:
- net ll_oe: now also RN7.5 (R4.2); no longer RN7.4 (R4.1)
- net ll_pull_down: now also RN7.4 (R4.1); no longer RN7.5 (R4.2)

Commit message: nearing the end
Parts:
- removed TP4: TestPoint, TestPoint:TestPoint_Pad_D1.0mm, symbol Connector:TestPoint
Other:
- note added: "10k resistor networks"
- note added: "buttons"
- moved on the sheet: R5, R6, RN6, RN7, SW1, SW3

Commit message: progress
Parts:
- removed LED1: LED_Generic_RGB_RABG, coquette_footprints:E6CC1205RGBC3UDA, symbol PCM_LED_AKL:LED_Generic_RGB_RABG
- removed R5, R6: 1.5k, Resistor_SMD:R_0603_1608Metric, symbol Device:R_US
- removed RN1, RN2: 2*R33, Resistor_SMD:R_Array_Convex_2x0603, symbol PCM_Resistor_US_AKL:R_2x0402_Convex
- added D1: LED, PCM_LED_SMD_AKL:LED_0603_1608Metric, symbol Device:LED
- added R8: R620, Resistor_SMD:R_0603_1608Metric, symbol Device:R_US
- added RN8: R33*4, PCM_Resistor_SMD_AKL:R_Array_Convex_4x0603, symbol PCM_Resistor_US_AKL:R_4x0603_Convex
- added RN9: 2*2.2k, Resistor_SMD:R_Array_Convex_2x0603, symbol PCM_Resistor_US_AKL:R_2x0402_Convex
Connections:
- net stat_blue is gone; now on net GND: RN6.2 (R2.1)
- net stat_green is gone; now on net GND: RN6.4 (R4.1)
- net stat_red is gone; now on net ll_pull_down: RN6.3 (R3.1)
- net GND: now also RN7.6 (R3.2); no longer RN7.7 (R2.2)
- net VBUS: now also RN7.4 (R4.1)
- net VCC: now also RN7.7 (R2.2), R8.2; no longer RN7.6 (R3.2)
- net VDC: now also RN6.8 (R1.2); no longer RN6.1 (R1.1)
- net ch1: now also MDBT1.7 (P0.26/AIN5); no longer MDBT1.56 (P0.31)
- net ch10: now also MDBT1.45 (P1.00); no longer MDBT1.27 (P0.14/QSPI1)
- net ch11: now also MDBT1.43 (P1.01); no longer MDBT1.26 (P0.17/QSPI_SCK)
- net ch12: now also MDBT1.39 (P0.05/AIN1); no longer MDBT1.23 (P0.15/QSPI2)
- net ch13: now also MDBT1.35 (P0.06/AIN2); no longer MDBT1.25 (P0.22)
- net ch14: now also MDBT1.12 (P0.21); no longer MDBT1.22 (P1.05)
- net ch15: now also MDBT1.13 (P0.20); no longer MDBT1.21 (P0.13/QSPI0)
- net ch16: now also MDBT1.14 (P0.19); no longer MDBT1.20 (P0.07/AIN3)
- net ch17: now also MDBT1.16 (P0.18/QSPI_CSN); no longer MDBT1.9 (P0.25/AIN4)
- net ch18: now also MDBT1.28 (P0.16/QSPI3); no longer MDBT1.7 (P0.26/AIN5)
- net ch19: now also MDBT1.27 (P0.14/QSPI1); no longer MDBT1.16 (P0.18/QSPI_CSN)
- net ch2: now also MDBT1.9 (P0.25/AIN4); no longer MDBT1.55 (P1.11)
- net ch20: now also MDBT1.26 (P0.17/QSPI_SCK); no longer MDBT1.14 (P0.19)
- net ch21: now also MDBT1.23 (P0.15/QSPI2); no longer MDBT1.13 (P0.20)
- net ch22: now also MDBT1.25 (P0.22); no longer MDBT1.12 (P0.21)
- net ch23: now also MDBT1.21 (P0.13/QSPI0); no longer MDBT1.11 (P1.04)
- net ch24: now also MDBT1.22 (P1.05); no longer MDBT1.10 (P1.06)
- net ch3: now also MDBT1.57 (P0.30); no longer MDBT1.51 (P1.13)
- net ch4: now also MDBT1.56 (P0.31); no longer MDBT1.49 (P1.14)
- net ch5: now also MDBT1.55 (P1.11); no longer MDBT1.45 (P1.00)
- net ch6: now also MDBT1.53 (P1.12); no longer MDBT1.43 (P1.01)
- net ch7: now also MDBT1.51 (P1.13); no longer MDBT1.47 (P1.15)
- net ch8: now also MDBT1.49 (P1.14); no longer MDBT1.53 (P1.12)
- net ch9: now also MDBT1.47 (P1.15); no longer MDBT1.28 (P0.16/QSPI3)
- net chg_pg: now also MDBT1.63 (P1.07); no longer MDBT1.3 (P1.08)
- net chg_stat: now also MDBT1.64 (P1.09); no longer MDBT1.8 (P0.24)
- net disp: now also RN7.2 (R2.1); no longer RN7.3 (R3.1)
- net eepy: now also MDBT1.3 (P1.08), RN9.4 (R1.2); no longer MDBT1.57 (P0.30)
- net ext_on: now also MDBT1.62 (P0.23); no longer MDBT1.5 (P0.27/AIN6)
- net extcomin: now also RN7.3 (R3.1); no longer RN7.2 (R2.1)
- net gpio2: now also MDBT1.37 (P0.04/AIN0); no longer MDBT1.35 (P0.06/AIN2)
- net ll_oe: now also RN6.6 (R3.2); no longer RN7.5 (R4.2)
- net ll_pull_down: no longer RN7.4 (R4.1)
- net reset: now also RN9.3 (R2.2)
- net scl: now also RN8.3 (R3.1)
- net sda: now also RN8.4 (R4.1)
- net swdclk: now also RN8.1 (R1.1)
- net swdio: now also RN8.2 (R2.1)
- net vcc_en: now also RN6.1 (R1.1); no longer RN6.8 (R1.2)
- net at SW3.1: now also RN9.1 (R1.1)
- net at SW1.1: now also RN9.2 (R2.1)
- net swdio_nrf: now reaches MDBT1.4 (SWDIO)
- net swdio_nrf: now also RN8.7 (R2.2)
- net swdclk_nrf: now reaches MDBT1.2 (SWDCLK)
- net swdclk_nrf: now also RN8.8 (R1.2)
- net sda_nrf: now reaches MDBT1.33 (P1.02/TWI)
- net sda_nrf: now also RN8.5 (R4.2)
- net scl_nrf: now reaches MDBT1.31 (P1.03/TWI)
- net scl_nrf: now also RN8.6 (R3.2)
- net status_led_blue renamed bat_ts
- net bat_ts: no longer MDBT1.62 (P0.23)
- removed net status_led_green: MDBT1.63 (P1.07), RN6.6 (R3.2)
- net status_led_red renamed vcc_mode
- net vcc_mode: no longer MDBT1.64 (P1.09)
- new net: D1.2 (A), R8.1
- new net USB_ST: RN7.5 (R4.2)
- new net sp/ce cs: MDBT1.5 (P0.27/AIN6)
- new net sp/ce pwm: MDBT1.20 (P0.07/AIN3)
- new net status_led: D1.1 (K), MDBT1.8 (P0.24)
- no-connect marks 5 -> 4
Other:
- note added: "resistor networks"
- note removed: "10k resistor networks"
- moved on the sheet: C18, C19, C49, L2, L3

Commit message: new dcdc
Connections:
- net BATT_READ_EN: no longer names the net of MDBT1.59 (P1.10)
Changed lines of the file:
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@@
-		)
-	)
-	(global_label "BATT_READ_EN"
-		(shape input)
-		(at 120.65 58.42 0)
-		(fields_autoplaced yes)
-		(effects
-			(font
-				(size 1.27 1.27)
-			)
-			(justify left)
-		)
-		(property "Intersheetrefs" "${INTERSHEET_REFS}"
-			(at 134.4455 58.42 0)
-			(effects
-				(font
-					(size 1.27 1.27)
-				)
-				(justify left)
-				(hide yes)
-			)
 		)
 	)

Commit message: tweaks
Parts:
- C48, C49: footprint Capacitor_SMD:C_0603_1608Metric -> Capacitor_SMD:C_1206_3216Metric
- R21: footprint Resistor_SMD:R_0603_1608Metric -> Resistor_SMD:R_0805_2012Metric
Changed lines of the file:
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@@
 			)
 		)
-		(property "Footprint" "Resistor_SMD:R_0603_1608Metric"
+		(property "Footprint" "Resistor_SMD:R_0805_2012Metric"
 			(at 150.876 100.584 90)
 			(effects
@@
 			)
 		)
-		(property "Footprint" "Capacitor_SMD:C_0603_1608Metric"
+		(property "Footprint" "Capacitor_SMD:C_1206_3216Metric"
 			(at 110.7948 128.27 0)
 			(effects
@@
 			)
 		)
-		(property "Footprint" "Capacitor_SMD:C_0603_1608Metric"
+		(property "Footprint" "Capacitor_SMD:C_1206_3216Metric"
 			(at 145.0848 104.14 0)
 			(effects
