File: addons.kicad_sch (KiCad schematic)
At the start: 7 parts, among them J8 Conn_01x04_MountingPin, J9 Conn_02x03_Odd_Even

Commit message: nearing the end
Parts:
- removed C10: 1uF, Capacitor_SMD:C_0603_1608Metric, symbol Device:C
- removed FB5: 120 Ohm, PCM_Ferrite_SMD_AKL:Ferrite_0603_1608Metric, symbol PCM_Device_AKL:Ferrite_Bead
- removed R17: R2.2, Resistor_SMD:R_0603_1608Metric, symbol Device:R_US
- C12: value 10nF -> 0.1uF
Connections:
- net PRI_MID is gone; now on net VCC: C12.1 (+), J8.2 (Pin_2), J9.1 (Pin_1)

Commit message: progress
Parts:
- added J5: Conn_01x08_MountingPin, Connector_JST:JST_SH_SM08B-SRSS-TB_1x08-1MP_P1.00mm_Horizontal, symbol Connector_Generic_MountingPin:Conn_01x08_MountingPin
Connections:
- net GND: now also J5.1 (Pin_1), J5.MP (MountPin)
- net VCC: now also J5.7 (Pin_7)
- new net VDC: J5.8 (Pin_8)
- new net miso: J5.3 (Pin_3)
- new net mosi: J5.4 (Pin_4)
- new net sck: J5.5 (Pin_5)
- new net sp/ce cs: J5.6 (Pin_6)
- new net sp/ce pwm: J5.2 (Pin_2)
Other:
- note added: "sp/ce"
- moved on the sheet: C12, J8
