File: argb.kicad_sch (KiCad schematic)
At the start: 16 parts, among them J2 Conn_01x03_MountingPin, U4 TPS22917DBV, U7 SN74LV1T125DCK

Commit message: title page 3 of schematic
Other:
- title: (none) -> coquette mariposa argb
Changed lines of the file:
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@@
 	(paper "A4")
 	(title_block
+		(title "coquette mariposa argb")
 		(date "2025-02-02")
 		(rev "2.0")

Commit message: final to order
Connections:
- net GND: now also D15.3 (GND), D16.3 (GND), D17.3 (GND), D18.3 (GND); no longer D15.1 (VSS), D16.1 (VSS), D17.1 (VSS), D18.1 (VSS)
- net PRI_LO: now also D15.1 (VDD), D16.1 (VDD), D17.1 (VDD), D18.1 (VDD); no longer D15.3 (VDD), D16.3 (VDD), D17.3 (VDD), D18.3 (VDD)
- net argb_data: now also D15.4 (DIN); no longer D15.2 (DIN)
- net argb_data_out: now also D18.2 (DOUT); no longer D18.4 (DOUT)
- net at D17.2 (DOUT): now also D18.4 (DIN); no longer D16.4 (DOUT)
- net at D17.4 (DIN): now also D16.2 (DOUT); no longer D18.2 (DIN)
- new net: D15.2 (DOUT), D16.4 (DIN)
Other:
- moved on the sheet: C15, C16, C17, D16, D17, D18

Commit message: cleanup
Parts:
- added JP5: SolderJumper_2_Bridged, Jumper:SolderJumper-2_P1.3mm_Bridged_RoundedPad1.0x1.5mm, symbol Jumper:SolderJumper_2_Bridged
- added JP6: SolderJumper_3_Bridged12, Jumper:SolderJumper-3_P1.3mm_Bridged12_RoundedPad1.0x1.5mm, symbol Jumper:SolderJumper_3_Bridged12
- added R14: 10k, Resistor_SMD:R_0603_1608Metric, symbol Device:R_US
Connections:
- net GND: now also JP5.2 (B); no longer R18.1
- net VDC: now also R14.2
- net ext_on: now also JP6.1 (A); no longer U4.3 (ON)
- new net: JP5.1 (A), R18.1
- new net: JP6.3 (B), R14.1
- new net: JP6.2 (C), U4.3 (ON)
Other:
- moved on the sheet: C11, C13, C14, C15, C16, C17, C8, C9, D15, D16, D17, D18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

Commit message: v3 efforts
Parts:
- removed C13: 4.7uF, Capacitor_SMD:C_0603_1608Metric, symbol Device:C
- removed JP6: SolderJumper_3_Bridged12, Jumper:SolderJumper-3_P1.3mm_Bridged12_RoundedPad1.0x1.5mm, symbol Jumper:SolderJumper_3_Bridged12
- removed R14, R18: 10k, Resistor_SMD:R_0603_1608Metric, symbol Device:R_US
- added C13: 47uF, PCM_Capacitor_Tantalum_SMD_AKL:CP_EIA-3528-12_Kemet-T, symbol PCM_Capacitor_AKL:CP_SMD_Tantalum_Kemet-T_3528
- added C20, C21, C22, C23: 0.1uF, Capacitor_SMD:C_0603_1608Metric, symbol Device:C
- added D19, D20, D21, D22: SK6805-EC14, coquette_footprints:SK6805-EC14, symbol coquette_symbols:SK6805-EC14
- added R13: R620, Resistor_SMD:R_0603_1608Metric, symbol Device:R_US
- C11, C14, C15, C16, C17: footprint Capacitor_SMD:C_0402_1005Metric -> Capacitor_SMD:C_0603_1608Metric
- C8: value 10 uF -> 10uF
- C9: value 220pF -> 390pF
Connections:
- net GND: now also C13.2, C20.1, C21.1, C22.1, C23.1, D19.3 (GND), D20.3 (GND), D21.3 (GND), D22.3 (GND)
- net PRI_LO: now also C13.1, C20.2, C21.2, C22.2, C23.2, D19.1 (VDD), D20.1 (VDD), D21.1 (VDD), D22.1 (VDD)
- net argb_data_out: now also R13.1; no longer D18.2 (DOUT)
- net ext_on: now also U4.3 (ON)
- net ll_pull_down: now reaches JP5.1 (A)
- net ll_oe: now reaches U7.1 (~{OE})
- new net: D20.2 (DOUT), D21.4 (DIN)
- new net: D19.2 (DOUT), D20.4 (DIN)
- new net: D21.2 (DOUT), D22.4 (DIN)
- new net: D22.2 (DOUT), R13.2

Commit message: more rounding
Connections:
- net at D19.4 (DIN): now also D18.2 (DOUT)
Changed lines of the file:
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@@
+	(wire
+		(pts
+			(xy 116.84 91.44) (xy 128.27 91.44)
+		)
+		(stroke
+			(width 0)
+			(type default)
+		)
+	)
 	(wire
 		(pts

Commit message: nearing the end
Parts:
- C8: value 10uF -> 1uF
Other:
- moved on the sheet: J2
Changed lines of the file:
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@@
 	)
 	(rectangle
-		(start 155.575 22.225)
-		(end 194.945 48.895)
+		(start 146.685 21.59)
+		(end 179.07 48.895)
 		(stroke
 			(width 0)
@@
 	(rectangle
 		(start 19.05 74.295)
-		(end 269.875 106.68)
+		(end 242.57 106.68)
 		(stroke
 			(width 0)
@@
 	(rectangle
 		(start 68.58 21.59)
-		(end 151.765 52.07)
+		(end 144.145 52.07)
 		(stroke
 			(width 0)
@@
 	(text "argb out\n"
 		(exclude_from_sim no)
-		(at 159.512 21.336 0)
+		(at 150.622 20.574 0)
 		(effects
 			(font
@@
 	(wire
 		(pts
-			(xy 133.35 34.29) (xy 138.43 34.29)
-		)
-		(stroke
-			(width 0)
-			(type default)
-		)
-	)
-	(wire
-		(pts
 			(xy 82.55 76.2) (xy 109.22 76.2)
 		)
@@
 		)
 	)
+	(wire
+		(pts
+			(xy 148.59 31.75) (xy 165.1 31.75)
+		)
+		(stroke
+			(width 0)
+			(type default)
+		)
+	)
 	(global_label "argb_data"
 		(shape input)
@@
 	(global_label "argb_data_out"
 		(shape input)
-		(at 173.99 29.21 180)
+		(at 165.1 29.21 180)
 		(fields_autoplaced yes)
 		(effects
@@
 		)
 		(property "Intersheetrefs" "${INTERSHEET_REFS}"
-			(at 159.2751 29.21 0)
+			(at 150.3851 29.21 0)
 			(effects
 				(font
@@
 	(symbol
 		(lib_id "power:Earth")
-		(at 173.99 34.29 0)
+		(at 165.1 34.29 0)
 		(unit 1)
 		(exclude_from_sim no)
@@
 		(dnp no)
 		(property "Reference" "#PWR014"
-			(at 173.99 40.64 0)
+			(at 165.1 40.64 0)
 			(effects
 				(font
@@
 		)
 		(property "Value" "GND"
-			(at 172.466 38.862 0)
+			(at 163.576 38.862 0)
 			(effects
 				(font
@@
 		)
 		(property "Footprint" ""
-			(at 173.99 34.29 0)
+			(at 165.1 34.29 0)
 			(effects
 				(font
@@
 		)
 		(property "Datasheet" "~"
-			(at 173.99 34.29 0)
+			(at 165.1 34.29 0)
 			(effects
 				(font
@@
 		)
 		(property "Description" "Power symbol creates a global label with name \"Earth\""
-			(at 173.99 34.29 0)
+			(at 165.1 34.29 0)
 			(effects
 				(font
@@
 			)
 		)
-		(property "Value" "10uF"
+		(property "Value" "1uF"
 			(at 81.28 39.3699 0)
 			(effects
@@
 	)
 	(symbol
-		(lib_id "power:Earth")
-		(at 135.89 99.06 0)
-		(unit 1)
-		(exclude_from_sim no)
-		(in_bom yes)
-		(on_board yes)
-		(dnp no)
-		(fields_autoplaced yes)
-		(property "Reference" "#PWR0116"
-			(at 135.89 105.41 0)
-			(effects
-				(font
-					(size 1.27 1.27)
-				)
-				(hide yes)
-			)
-		)
-		(property "Value" "GND"
-			(at 135.89 104.14 0)
-			(effects
-				(font
-					(size 1.27 1.27)
-				)
-			)
-		)
-		(property "Footprint" ""
-			(at 135.89 99.06 0)
-			(effects
-				(font
-					(size 1.27 1.27)
-				)
-				(hide yes)
-			)
-		)
-		(property "Datasheet" "~"
-			(at 135.89 99.06 0)
-			(effects
-				(font
-					(size 1.27 1.27)
-				)
-				(hide yes)
-			)
-		)
-		(property "Description" "Power symbol creates a global label with name \"Earth\""
-			(at 135.89 99.06 0)
-			(effects
-				(font
-					(size 1.27 1.27)
-				)
-				(hide yes)
-			)
-		)
-		(pin "1"
-		)
-		(instances
-			(project "mariposa"
-				(path "/88abd3ac-3560-486a-811e-4281250949a6/3ca3d760-5559-4665-8ed1-eaf6a9f1daf8"
-					(reference "#PWR0116")
-					(unit 1)
-				)
-			)
-		)
-	)
-	(symbol
 		(lib_id "power:VDC")
 		(at 77.47 34.29 90)
@@
 	(symbol
 		(lib_id "power:PRI_LO")
-		(at 173.99 31.75 90)
-		(mirror x)
+		(at 148.59 31.75 0)
+		(mirror y)
 		(unit 1)
 		(exclude_from_sim no)
@@
 		(dnp no)
 		(property "Reference" "#PWR05"
-			(at 177.8 31.75 0)
+			(at 148.59 35.56 0)
 			(effects
 				(font
@@
 		)
 		(property "Value" "PRI_LO"
-			(at 167.64 31.75 90)
+			(at 148.59 25.4 90)
 			(effects
 				(font
@@
 		)
 		(property "Footprint" ""
-			(at 173.99 31.75 0)
+			(at 148.59 31.75 0)
 			(effects
 				(font
@@
 		)
 		(property "Datasheet" ""
-			(at 173.99 31.75 0)
+			(at 148.59 31.75 0)
 			(effects
 				(font
@@
 		)
 		(property "Description" "Power symbol creates a global label with name \"PRI_LO\""
-			(at 173.99 31.75 0)
+			(at 148.59 31.75 0)
 			(effects
 				(font
@@
 	(symbol
 		(lib_id "Connector_Generic_MountingPin:Conn_01x03_MountingPin")
-		(at 179.07 31.75 0)
+		(at 170.18 31.75 0)
 		(unit 1)
 		(exclude_from_sim no)
@@
 		(dnp no)
 		(property "Reference" "J2"
-			(at 178.054 25.908 0)
+			(at 169.164 25.908 0)
 			(effects
 				(font
@@
 		)
 		(property "Value" "Conn_01x03_MountingPin"
-			(at 184.404 45.212 90)
+			(at 175.514 45.212 90)
 			(effects
 				(font
@@
 		)
 		(property "Footprint" "Connector_JST:JST_SH_SM03B-SRSS-TB_1x03-1MP_P1.00mm_Horizontal"
-			(at 179.07 31.75 0)
+			(at 170.18 31.75 0)
 			(effects
 				(font
@@
 		)
 		(property "Datasheet" "~"
-			(at 179.07 31.75 0)
+			(at 170.18 31.75 0)
 			(effects
 				(font
@@
 		)
 		(property "Description" "Generic connectable mounting pin connector, single row, 01x03, script generated (kicad-library-utils/schlib/autogen/connector/)"
-			(at 179.07 31.75 0)
+			(at 170.18 31.75 0)
 			(effects
 				(font
@@
 	(symbol
 		(lib_id "power:Earth")
-		(at 179.07 39.37 0)
+		(at 170.18 39.37 0)
 		(unit 1)
 		(exclude_from_sim no)
@@
 		(dnp no)
 		(property "Reference" "#PWR062"
-			(at 179.07 45.72 0)
+			(at 170.18 45.72 0)
 			(effects
 				(font
@@
 		)
 		(property "Value" "GND"
-			(at 177.8 43.688 0)
+			(at 168.91 43.688 0)
 			(effects
 				(font
@@
 		)
 		(property "Footprint" ""
-			(at 179.07 39.37 0)
+			(at 170.18 39.37 0)
 			(effects
 				(font
@@
 		)
 		(property "Datasheet" "~"
-			(at 179.07 39.37 0)
+			(at 170.18 39.37 0)
 			(effects
 				(font
@@
 		)
 		(property "Description" "Power symbol creates a global label with name \"Earth\""
-			(at 179.07 39.37 0)
+			(at 170.18 39.37 0)
 			(effects
 				(font
@@
 	(symbol
 		(lib_id "power:PRI_LO")
-		(at 138.43 34.29 270)
+		(at 133.35 34.29 0)
 		(unit 1)
 		(exclude_from_sim no)
@@
 		(fields_autoplaced yes)
 		(property "Reference" "#PWR0110"
-			(at 134.62 34.29 0)
+			(at 133.35 38.1 0)
 			(effects
 				(font
@@
 		)
 		(property "Value" "PRI_LO"
-			(at 142.24 34.2899 90)
+			(at 133.35 29.21 0)
 			(effects
 				(font
 					(size 1.27 1.27)
 				)
-				(justify left)
 			)
 		)
 		(property "Footprint" ""
-			(at 138.43 34.29 0)
+			(at 133.35 34.29 0)
 			(effects
 				(font
@@
 		)
 		(property "Datasheet" ""
-			(at 138.43 34.29 0)
+			(at 133.35 34.29 0)
 			(effects
 				(font
@@
 		)
 		(property "Description" "Power symbol creates a global label with name \"PRI_LO\""
-			(at 138.43 34.29 0)
+			(at 133.35 34.29 0)
 			(effects
 				(font

Commit message: progress
Parts:
- removed C13: 47uF, PCM_Capacitor_Tantalum_SMD_AKL:CP_EIA-3528-12_Kemet-T, symbol PCM_Capacitor_AKL:CP_SMD_Tantalum_Kemet-T_3528
- removed C22, C23: 0.1uF, Capacitor_SMD:C_0603_1608Metric, symbol Device:C
- removed D21, D22: SK6805-EC14, coquette_footprints:SK6805-EC14, symbol coquette_symbols:SK6805-EC14
- added C53: 10uF, Capacitor_SMD:C_0603_1608Metric, symbol Device:C
Connections:
- net GND: now also C53.2
- net PRI_LO: now also C53.1
- net at D20.2 (DOUT): now also R13.2
Other:
- moved on the sheet: R13

Commit message: tweaks
Parts:
- C53: footprint Capacitor_SMD:C_0603_1608Metric -> Capacitor_SMD:C_0805_2012Metric
Changed lines of the file:
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@@
 			)
 		)
-		(property "Footprint" "Capacitor_SMD:C_0603_1608Metric"
+		(property "Footprint" "Capacitor_SMD:C_0805_2012Metric"
 			(at 132.3848 41.91 0)
 			(effects
