File: argb.kicad_sch (KiCad schematic)
At the start: 21 parts, among them J2 Conn_01x03_MountingPin, U4 TPS22917DBV, U7 SN74LV1T125DCK

Commit message: fixes
Parts:
- R13: footprint Resistor_SMD:R_0603_1608Metric -> Resistor_SMD:R_0805_2012Metric
Changed lines of the file:
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@@
 			)
 		)
-		(property "Footprint" "Resistor_SMD:R_0603_1608Metric"
+		(property "Footprint" "Resistor_SMD:R_0805_2012Metric"
 			(at 169.164 94.996 90)
 			(effects
