File: power.kicad_sch (KiCad schematic)
At the start: 36 parts, among them J4 USB_C_Receptacle_USB2.0_16P, U2 BQ25170DSGR, U3 LM66100DCK, U5 TPS628438DRL, U6 LM66100DCK

Commit message: final to order
Parts:
- added R8: 10k, Resistor_SMD:R_0603_1608Metric, symbol Device:R_US
Connections:
- net GND: no longer U6.5 (ST)
- net VBUS: now also R8.2; no longer U3.3 (~{CE})
- new net: R8.1, U3.3 (~{CE}), U6.5 (ST)
Changed lines of the file:
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@@
+		(color 0 0 0 0)
+	)
+	(junction
+		(at 195.58 93.98)
+		(diameter 0)
 		(color 0 0 0 0)
 	)
@@
 	(wire
 		(pts
+			(xy 252.73 93.98) (xy 195.58 93.98)
+		)
+		(stroke
+			(width 0)
+			(type default)
+		)
+	)
+	(wire
+		(pts
 			(xy 187.96 76.2) (xy 199.39 76.2)
 		)
@@
 	(wire
 		(pts
-			(xy 252.73 86.36) (xy 252.73 81.28)
+			(xy 195.58 81.28) (xy 199.39 81.28)
+		)
+		(stroke
+			(width 0)
+			(type default)
+		)
+	)
+	(wire
+		(pts
+			(xy 252.73 81.28) (xy 252.73 93.98)
 		)
 		(stroke
@@
 		(pts
 			(xy 50.8 38.1) (xy 55.88 38.1)
+		)
+		(stroke
+			(width 0)
+			(type default)
+		)
+	)
+	(wire
+		(pts
+			(xy 195.58 93.98) (xy 195.58 81.28)
 		)
 		(stroke
@@
 	(rectangle
 		(start 181.61 66.04)
-		(end 260.35 96.52)
+		(end 281.94 109.22)
 		(stroke
 			(width 0)
@@
 	(symbol
 		(lib_id "power:VBUS")
-		(at 199.39 81.28 90)
+		(at 195.58 101.6 180)
 		(unit 1)
 		(exclude_from_sim no)
@@
 		(dnp no)
 		(property "Reference" "#PWR086"
-			(at 203.2 81.28 0)
+			(at 195.58 97.79 0)
 			(effects
 				(font
@@
 		)
 		(property "Value" "VBUS"
-			(at 197.612 83.82 90)
+			(at 198.12 103.378 90)
 			(effects
 				(font
@@
 		)
 		(property "Footprint" ""
-			(at 199.39 81.28 0)
+			(at 195.58 101.6 0)
 			(effects
 				(font
@@
 		)
 		(property "Datasheet" ""
-			(at 199.39 81.28 0)
+			(at 195.58 101.6 0)
 			(effects
 				(font
@@
 		)
 		(property "Description" "Power symbol creates a global label with name \"VBUS\""
-			(at 199.39 81.28 0)
+			(at 195.58 101.6 0)
 			(effects
 				(font
@@
 	(symbol
 		(lib_id "power:Earth")
-		(at 252.73 86.36 0)
-		(unit 1)
-		(exclude_from_sim no)
-		(in_bom yes)
-		(on_board yes)
-		(dnp no)
-		(fields_autoplaced yes)
-		(property "Reference" "#PWR089"
-			(at 252.73 92.71 0)
-			(effects
-				(font
-					(size 1.27 1.27)
-				)
-				(hide yes)
-			)
-		)
-		(property "Value" "GND"
-			(at 252.73 91.44 0)
-			(effects
-				(font
-					(size 1.27 1.27)
-				)
-			)
-		)
-		(property "Footprint" ""
-			(at 252.73 86.36 0)
-			(effects
-				(font
-					(size 1.27 1.27)
-				)
-				(hide yes)
-			)
-		)
-		(property "Datasheet" "~"
-			(at 252.73 86.36 0)
-			(effects
-				(font
-					(size 1.27 1.27)
-				)
-				(hide yes)
-			)
-		)
-		(property "Description" "Power symbol creates a global label with name \"Earth\""
-			(at 252.73 86.36 0)
-			(effects
-				(font
-					(size 1.27 1.27)
-				)
-				(hide yes)
-			)
-		)
-		(pin "1"
-		)
-		(instances
-			(project "mariposa"
-				(path "/88abd3ac-3560-486a-811e-4281250949a6/aefb2378-1b2c-46d5-9c89-47f5f798e766"
-					(reference "#PWR089")
-					(unit 1)
-				)
-			)
-		)
-	)
-	(symbol
-		(lib_id "power:Earth")
 		(at 196.85 52.07 0)
 		(unit 1)
@@
 					(unit 1)
 				)
+			)
+		)
+	)
+	(symbol
+		(lib_id "Device:R_US")
+		(at 195.58 97.79 0)
+		(unit 1)
+		(exclude_from_sim no)
+		(in_bom yes)
+		(on_board yes)
+		(dnp no)
+		(property "Reference" "R8"
+			(at 198.628 97.79 90)
+			(effects
+				(font
+					(size 1.27 1.27)
+				)
+			)
+		)
+		(property "Value" "10k"
+			(at 200.406 97.79 90)
+			(effects
+				(font
+					(size 1.27 1.27)
+				)
+			)
+		)
+		(property "Footprint" "Resistor_SMD:R_0603_1608Metric"
+			(at 196.596 98.044 90)
+			(effects
+				(font
+					(size 1.27 1.27)
+				)
+				(hide yes)
+			)
+		)
+		(property "Datasheet" "~"
+			(at 195.58 97.79 0)
+			(effects
+				(font
+					(size 1.27 1.27)
+				)
+				(hide yes)
+			)
+		)
+		(property "Description" "Resistor, US symbol"
+			(at 195.58 97.79 0)
+			(effects
+				(font
+					(size 1.27 1.27)
+				)
+				(hide yes)
+			)
+		)
+		(pin "2"
+		)
+		(pin "1"
+		)
+		(instances
+			(project "mariposa"
+				(path "/88abd3ac-3560-486a-811e-4281250949a6/aefb2378-1b2c-46d5-9c89-47f5f798e766"
+					(reference "R8")
+					(unit 1)
+				)

Commit message: cleanup
Parts:
- added JP2: SolderJumper_2_Bridged, Jumper:SolderJumper-2_P1.3mm_Bridged_RoundedPad1.0x1.5mm, symbol Jumper:SolderJumper_2_Bridged
Connections:
- net VBUS: now also R8.1; no longer R8.2
- net VDC: now also JP2.1 (A); no longer U5.4 (EN)
- net USB_ST: now reaches U3.3 (~{CE}), U6.5 (ST)
- net USB_ST: now also R8.2; no longer R8.1
- new net: JP2.2 (B), U5.4 (EN)
Other:
- moved on the sheet: C44, C45, C6, C7, L1, R10, R11, R8, R9, U3, U5, U6

Commit message: v3 efforts
Parts:
- removed D11, D14, D2, D3, D4, D7, D8: TPD4E1U06, coquette_footprints:TPD4E1U06, symbol coquette_symbols:TPD4E1U06
- removed R8: 10k, Resistor_SMD:R_0603_1608Metric, symbol Device:R_US
- removed U5: TPS628438DRL, coquette_footprints:TPS628438DRL, symbol Regulator_Switching:TPS628438DRL
- added R14, R16: 10k, Resistor_SMD:R_0603_1608Metric, symbol Device:R_US
- added U1: TPS62840DLC, Package_SON:Texas_VSON-HR-8_1.5x2mm_P0.5mm, symbol coquette_symbols:TPS62840DLC
- C4, C5: footprint Capacitor_SMD:C_0402_1005Metric -> Capacitor_SMD:C_0603_1608Metric
- C44: value 4.7 uF -> 4.7uF
- C45: value 10 uF -> 10uF
- L1: value 1 uH -> 2.2uH; footprint Inductor_SMD:L_0603_1608Metric -> Inductor_SMD:L_1008_2520Metric
- R10: value 2M -> 1.5M
- R11: value 249k -> 52.3k
- R9: value 787k -> 750k
Connections:
- net +BATT: now also BT1.2 (Pin_2); no longer BT1.1 (Pin_1)
- net GND: now also BT1.1 (Pin_1), R16.1, U1.1 (GND); no longer BT1.2 (Pin_2)
- net PRI_MID: now also D12.3 (L2); no longer D12.1 (L1)
- net USB_ST: now also R14.2
- net VBUS: now also R14.1
- net VCC: now also D13.3 (L2), U1.8 (VOS); no longer D13.1 (L1)
- net VDC: now also U1.2 (VIN); no longer JP2.1 (A)
- net reset: now also D13.1 (L1); no longer D13.6 (L4)
- net sda: now also D12.1 (L1); no longer D12.3 (L2)
- net swdclk: now also D13.6 (L4); no longer D13.4 (L3)
- net swdio: now also D13.4 (L3); no longer D13.3 (L2)
- net at R11.1: now also U1.5 (VSET)
- net vcc_en: now reaches JP2.2 (B)
- net SW: now reaches L1.1 (+)
- net SW: now also U1.7 (SW)
- new net: R16.2, U1.3 (MODE)
- new net: JP2.1 (A), U1.4 (EN)
- no-connect marks 2 -> 3
Other:
- note added: "R11 – use 52.3k for 3V, 267k for 3V3"
- moved on the sheet: C44, C45, JP2, L1, R11

Commit message: nearing the end
Connections:
- net PRI_MID is gone; now on net gpio2: D12.3 (L2)
- net VCC: now also D10.4 (L3)
- net gpio2: no longer D10.4 (L3)
- net gpio1: no longer names the net of D10.3 (L2)
Other:
- moved on the sheet: C6, C7, R14, U3, U6

Commit message: progress
Parts:
- removed R12, R14, R16: 10k, Resistor_SMD:R_0603_1608Metric, symbol Device:R_US
- added D14: TPD4E1U06, coquette_footprints:TPD4E1U06, symbol coquette_symbols:TPD4E1U06
- R15: value 27k -> 36k
- R7: value 1.5k -> 1.8k
Connections:
- net GND: now also D14.2 (VN), D14.5 (NC)
- net VCC: no longer D10.4 (L3)
- net argb_data_out: now also D10.4 (L3); no longer D12.6 (L4)
- net gpio2: now also D10.3 (L2); no longer D12.3 (L2)
- net sda: now also D12.3 (L2); no longer D12.1 (L1)
- net bat_ts: now reaches U2.3 (TS)
- net vcc_mode: now reaches U1.3 (MODE)
- new net miso: D14.3 (L2)
- new net mosi: D14.1 (L1)
- new net sck: D14.6 (L4)
- new net sp/ce cs: D12.6 (L4)
- new net sp/ce pwm: D12.1 (L1)
Other:
- note added: "R10 – enter as 1.614 in ZMK config (so it thinks 4.1V is 4.2)"
- moved on the sheet: BT1, C44, C45, C46, C47, C6, C7, D10, D12, D13, JP2, L1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

Commit message: new dcdc
Parts:
- removed U1: TPS62840DLC, Package_SON:Texas_VSON-HR-8_1.5x2mm_P0.5mm, symbol coquette_symbols:TPS62840DLC
- added C10: 10nF, Capacitor_SMD:C_0603_1608Metric, symbol PCM_Elektuur:C
- added U1: TPS62842DGRR, Package_SO:HVSSOP-8-1EP_3x3mm_P0.65mm_EP1.57x1.89mm_ThermalVias, symbol mariposa:TPS62842DGRR
- JP2: value SolderJumper_2_Bridged -> Jumper
- R10: value 1.5M -> 15M; footprint Resistor_SMD:R_0603_1608Metric -> Resistor_SMD:R_1206_3216Metric
- R11: value 52.3k -> 28.7k
- R9: value 750k -> 7.5M
Connections:
- net BATT_READ_EN is gone; now on net BATT_READ: R10.2
- net +BATT: now also R9.2; no longer R9.1
- net BATT_READ: now also R9.1, C10.1 (+); no longer R10.1, R9.2
- net GND: now also R10.1, C10.2 (-), U1.8 (GND), U1.9 (GND)
- net SW: now also L1.2 (-), U1.2 (SW); no longer L1.1 (+)
- net VCC: now also L1.1 (+), U1.1 (VOS); no longer L1.2 (-)
- net VDC: now also U1.6 (VIN)
- net vcc_mode: now also U1.3 (MODE)
- net at JP2.1 (A): now also U1.5 (EN)
- net at R11.1: now also U1.4 (VSET)
Other:
- note added: "R11 – 28.7k is 3.1V, use 52.3k for 3.3V, 21.5k for 3V"
- note removed: "R11 – use 52.3k for 3V, 267k for 3V3"
- moved on the sheet: C44, C45, JP2, L1, R10, R11, R9

Commit message: tweaks
Parts:
- C44: footprint Capacitor_SMD:C_0603_1608Metric -> Capacitor_SMD:C_1206_3216Metric
- C45: footprint Capacitor_SMD:C_0603_1608Metric -> Capacitor_SMD:C_0805_2012Metric
Changed lines of the file:
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@@
 		(length 2.54)
 		(shape diamond)
-		(at 179.07 35.56 90)
-		(effects
-			(font
-				(size 1.27 1.27)
-			)
-			(justify left bottom)
-		)
-		(property "Netclass" "power"
-			(at 176.53 42.164 90)
-			(effects
-				(font
-					(size 1.27 1.27)
-					(italic yes)
-				)
-				(justify left)
-			)
-		)
-	)
-	(netclass_flag ""
-		(length 2.54)
-		(shape diamond)
 		(at 50.8 38.1 180)
 		(effects
@@
 			)
 		)
-		(property "Footprint" "Capacitor_SMD:C_0603_1608Metric"
+		(property "Footprint" "Capacitor_SMD:C_1206_3216Metric"
 			(at 247.3452 36.83 0)
 			(effects
@@
 			)
 		)
-		(property "Footprint" "Capacitor_SMD:C_0603_1608Metric"
+		(property "Footprint" "Capacitor_SMD:C_0805_2012Metric"
 			(at 188.9252 41.91 0)
 			(effects

Commit message: maybe order?
Parts:
- R9: footprint Resistor_SMD:R_0603_1608Metric -> Resistor_SMD:R_0805_2012Metric
Connections:
- net chg_pg: now also U2.5 (STAT); no longer U2.6 (PG_N)
- net chg_stat: now also U2.6 (PG_N); no longer U2.5 (STAT)
Other:
- note removed: "R10 – enter as 1.614 in ZMK config (so it thinks 4.1V is 4.2)"
Changed lines of the file:
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@@
-		)
-	)
-	(text "R10 – enter as 1.614 in ZMK config (so it thinks 4.1V is 4.2)"
-		(exclude_from_sim no)
-		(at 161.29 98.552 0)
-		(effects
-			(font
-				(size 1.27 1.27)
-			)
 		)
 	)
@@
 	(global_label "chg_pg"
 		(shape input)
+		(at 154.94 50.8 0)
+		(fields_autoplaced yes)
+		(effects
+			(font
+				(size 1.27 1.27)
+			)
+			(justify left)
+		)
+		(property "Intersheetrefs" "${INTERSHEET_REFS}"
+			(at 163.2191 50.8 0)
+			(effects
+				(font
+					(size 1.27 1.27)
+				)
+				(justify left)
+				(hide yes)
+			)
+		)
+	)
+	(global_label "chg_stat"
+		(shape input)
 		(at 154.94 43.18 0)
 		(fields_autoplaced yes)
@@
 		)
 		(property "Intersheetrefs" "${INTERSHEET_REFS}"
-			(at 163.2191 43.18 0)
-			(effects
-				(font
-					(size 1.27 1.27)
-				)
-				(justify left)
-				(hide yes)
-			)
-		)
-	)
-	(global_label "chg_stat"
-		(shape input)
-		(at 154.94 50.8 0)
-		(fields_autoplaced yes)
-		(effects
-			(font
-				(size 1.27 1.27)
-			)
-			(justify left)
-		)
-		(property "Intersheetrefs" "${INTERSHEET_REFS}"
-			(at 165.0579 50.8 0)
+			(at 165.0579 43.18 0)
 			(effects
 				(font
@@
 			)
 		)
-		(property "Footprint" "Resistor_SMD:R_0603_1608Metric"
+		(property "Footprint" "Resistor_SMD:R_0805_2012Metric"
 			(at 154.686 91.186 90)
 			(effects
